File: Rack_Display.kicad_pcb (KiCad board)
At the start: 2 copper layers, 122 x 41 mm, 116 parts, among them J1 5-104363-2, J2 5-104363-2, J3 5-104363-2, J4 5-104362-3, J5 Conn_01x20, J6 Conn_01x20, J7 Conn_01x08_Socket, J8 Conn_01x02, J9 5-104362-3, K1 G5V-1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

Commit message: "TME"
Parts:
- C5, C6: value 1uF/50V -> 1uF/10V
- D14, D16, D17, D5: value RED -> GREEN
- D3: value RED -> YELLOW
- F1: value Fuse_Small -> PTF78
- F2, F3, F4: value 30mA -> 50mA
- F5: value T1A -> PTF78
- R18, R50: value 1k -> 560R
- R21, R44: value 1k -> 4k7
- R22, R23, R26: value 10k -> 4k7
